Commit message: robot moving and mapping

File: luis/quadruped_description/urdf/ContinuO_lidar.xacro (robot description, xacro)
@@ -5,4 +5,9 @@
 <robot xmlns:xacro="http://ros.org/wiki/xacro" name="ContinuO">
   <xacro:include filename="$(find quadruped_description)/urdf/robot.gazebo"/>
+  <link name="base_link" />
+  <joint name="dummy_joint" type="fixed">
+    <parent link="base_link" />
+    <child link="base" />
+  </joint>
   <material name="orange">
     <color rgba="0.12 0.15 0.2 1.0"/>
@@ -1103,4 +1108,57 @@
     </plugin>
   </gazebo>
+  <gazebo reference="os_sensor">
+    <sensor type="ray" name="ouster_sensor">
+      <pose>0 0 0 0 0 0</pose>
+      <visualize>false</visualize>
+      <always_on>true</always_on>
+      <update_rate>10.0</update_rate>
+      <ray>
+        <scan>
+          <horizontal>
+            <samples>512</samples>
+            <resolution>1</resolution>
+            <min_angle>-3.14159265</min_angle>
+            <max_angle>3.14159265</max_angle>
+          </horizontal>
+          <vertical>
+            <samples>64</samples>
+            <resolution>1</resolution>
+            <min_angle>-0.261799</min_angle> <max_angle>0.261799</max_angle>
+          </vertical>
+        </scan>
+        <range>
+          <min>0.1</min>
+          <max>100.0</max>
+          <resolution>0.01</resolution>
+        </range>
+        <noise>
+          <type>gaussian</type>
+          <mean>0.0</mean>
+          <stddev>0.01</stddev>
+        </noise>
+      </ray>
+      <plugin name="gazebo_ros_laser_controller" filename="libgazebo_ros_velodyne_laser.so">
+        <topicName>/ouster/points</topicName>
+        <frameName>os_sensor</frameName>
+        <organize_cloud>false</organize_cloud>
+        <min_range>0.1</min_range>
+        <max_range>100.0</max_range>
+        <gaussianNoise>0.01</gaussianNoise>
+      </plugin>
+    </sensor>
+  </gazebo>
+  <gazebo>
+    <plugin name="ground_truth_odometry" filename="libgazebo_ros_p3d.so">
+      <alwaysOn>true</alwaysOn>
+      <bodyName>base_link</bodyName>
+      <updateRate>50.0</updateRate>
+      <topicName>/odom</topicName>
+      <gaussianNoise>0.01</gaussianNoise>
+      <frameName>world</frameName>
+      <xyzOffsets>0 0 0</xyzOffsets>
+      <rpyOffsets>0 0 0</rpyOffsets>
+    </plugin>
+  </gazebo>
 <transmission name="trans_FL_HAA">
   <type>transmission_interface/SimpleTransmission</type>

Commit message: changed lidar angles

File: luis/quadruped_description/urdf/ContinuO_lidar.xacro (robot description, xacro)
@@ -87,5 +87,5 @@
   </link>
   <joint name="base_to_lidar" type="fixed">
-    <origin xyz="0.27 0 0.05" rpy="0 45 0" />
+    <origin xyz="0.3 0 0.05" rpy="0 0.7854 0" />
     <parent link="base" />
     <child link="os_sensor" />
@@ -1119,15 +1119,15 @@
             <samples>512</samples>
             <resolution>1</resolution>
-            <min_angle>-3.14159265</min_angle>
-            <max_angle>3.14159265</max_angle>
+            <min_angle>-1.5708</min_angle>
+            <max_angle>1.5708</max_angle>
           </horizontal>
           <vertical>
             <samples>64</samples>
             <resolution>1</resolution>
-            <min_angle>-0.261799</min_angle> <max_angle>0.261799</max_angle>
+            <min_angle>-0.785398</min_angle> <max_angle>0.785398</max_angle>
           </vertical>
         </scan>
         <range>
-          <min>0.1</min>
+          <min>0.5</min>
           <max>100.0</max>
           <resolution>0.01</resolution>
